File: teensy-plus-2.kicad_pcb (KiCad board)
At the start: 2 copper layers, 30.5 x 38.1 mm, 36 parts, among them J1 Conn_01x03_Male, J10 Conn_01x14, J11 Conn_02x04_Odd_Even, J12 Conn_01x02, J2 Conn_01x03_Male, J3 Conn_01x14_Male, J4 Conn_01x03_Male, J5 Conn_01x05_Male, J6 Conn_01x03_Male, J7 Conn_01x14_Male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

Commit message: Updated to version 3.0
- Changed to 74AHCT125
- Removed 22 ohm resistors
- IO23 is now active low

Signed-off-by: Aaron Williams <aaron.w2@gmail.com>
Parts:
- removed C17, C18, C19, C20: 4700nF DNS, Capacitor_SMD:C_0603_1608Metric
- removed RN1: 22, Resistor_SMD:R_Array_Convex_4x0603
- added C1: 0.1uF, Capacitor_SMD:C_0603_1608Metric, F.Cu at (33.9, 57.9)
- U1: value TXB0104PWR -> SN74AHCT125N; footprint digikey-footprints:TSSOP-14_W4.4mm -> Package_DFN_QFN:Texas_S-PVQFN-N14
- moved J4 11.0 mm to (36.2, 62.4), turned to 270 degrees
- moved C2 10.8 mm to (36.0, 34.5)
- moved C4 9.72 mm to (37.2, 48.5), turned to 90 degrees
- moved J6 9.02 mm to (29.8, 53.3)
- moved C3 7.36 mm to (36.0, 36.0), turned to 180 degrees
- moved C1 6.81 mm to (30.8, 37.2)
- moved J1 6.35 mm to (29.8, 62.4), turned to 90 degrees
- moved C9 6.31 mm to (33.8, 48.0)
- moved D1 2.75 mm to (29.3, 46.0)
- moved C8 2.70 mm to (32.6, 45.6)
- moved C6 1.16 mm to (28.8, 49.2), turned to 0 degrees
- moved U1 0.94 mm to (35.4, 39.2), turned to 0 degrees
- moved J2 0.06 mm to (36.2, 53.4)
Connections:
- D1 pad 4: Net-(D1-Pad4) -> /DIN
- J1 pad 2: /IO0_HR -> /IO0_H
- J10 pad 2: /IO6_HR -> /IO6_H
- J10 pad 3: /IO5_HR -> /IO5_H
- J10 pad 4: /IO0_HR -> /IO0_H
- J2 pad 2: /IO5_HR -> /IO5_H
- J4 pad 2: /IO6_HR -> /IO6_H
- J6 pad 2: /DO_R -> /DO
- U1 pad 1: +3V3 -> /IO23
- U1 pad 10: Net-(D1-Pad4) -> /IO23
- U1 pad 11: /IO6_H -> /IO5_H
- U1 pad 12: /IO5_H -> /IO5
- U1 pad 13: /IO0_H -> /IO23
- U1 pad 3: /IO5 -> /IO0_H
- U1 pad 4: /IO6 -> /IO23
- U1 pad 6: Net-(U1-Pad6) -> /DIN
- U1 pad 8: /IO23 -> /IO6_H
- U1 pad 9: Net-(U1-Pad9) -> /IO6
Routing:
- net GND: track 70.6 -> 139.6 mm, vias 18 -> 49
- net /IO0_HR: track 33.4 -> 0.00 mm
- net /IO0_H: track 7.62 -> 39.6 mm, vias 1 -> 5
- net /DO_R: track 30.9 -> 0.00 mm, vias 3 -> 0
- net /IO6_H: track 9.14 -> 38.2 mm, vias 1 -> 3
- net /IO6_HR: track 28.9 -> 0.00 mm, vias 2 -> 0
- net /IO5_H: track 8.36 -> 36.0 mm, vias 1 -> 4
- net /IO5_HR: track 24.5 -> 0.00 mm, vias 1 -> 0
- net /IO23: track 11.8 -> 21.2 mm, vias 0 -> 5
- net /DIN: track 0.00 -> 8.96 mm, vias 0 -> 2
- net +5V: track 110.8 -> 106.6 mm, vias 7 -> 3
- net +3V3: track 76.6 -> 72.4 mm, vias 1 -> 4
- net /IO6: track 17.2 -> 13.6 mm
- net /IO0: track 4.99 -> 8.57 mm, vias 0 -> 2
- net /DO: track 3.26 -> 6.82 mm, vias 1 -> 0
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- added copper zone on F.Cu, net GND
- removed copper zone on F.Cu, net +5V
Other:
- board text added: "Revision 3.0"
- board text removed: "Revision 2.0"
