File: teensy-plus-2.sch (KiCad schematic (older format))
At the start: 35 parts, among them J1 Conn_01x03_Male, J10 Conn_01x14, J11 Conn_02x04_Odd_Even, J12 Conn_01x02, J2 Conn_01x03_Male, J3 Conn_01x14_Male, J4 Conn_01x03_Male, J5 Conn_01x05_Male, J6 Conn_01x03_Male, J7 Conn_01x14_Male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

Commit message: Updated to version 3.0
- Changed to 74AHCT125
- Removed 22 ohm resistors
- IO23 is now active low

Signed-off-by: Aaron Williams <aaron.w2@gmail.com>
Parts:
- removed C17, C18, C19, C20: 4700nF DNS, Capacitor_SMD:C_0603_1608Metric, symbol Device:C
- removed RN1: 22, Resistor_SMD:R_Array_Convex_4x0603, symbol Device:R_Pack04
- removed U1: TXB0104PWR, digikey-footprints:TSSOP-14_W4.4mm, symbol dk_Logic-Translators-Level-Shifters:TXB0104PWR
- added U1: SN74AHCT125N, Package_DFN_QFN:Texas_S-PVQFN-N14, symbol dk_Logic-Buffers-Drivers-Receivers-Transceivers:SN74AHCT125N
Connections:
- net labels added: DIN
- net labels removed: IO0_HR, IO5_HR, IO6_HR
- wire segments 146 -> 136
Other:
- moved on the sheet: D1
